File: KiCAD Files/ESP32 Waage.sch (KiCad schematic (older format))
At the start: 7 parts, among them SW1 SW_Reed, U1 BME280Socket, U2 ESP32WROVERSocket, U3 HX711Socket, U4 SupplSpringTerm, U5 DS18B20SpringTerm, U6 HX711SpringTerm

Commit message: dded resitors, capacitors, missing connections
Parts:
- added C1, C2, C3: C, symbol Device:C
- added R1, R2: R, symbol Device:R
Connections:
- wire segments 47 -> 83
- no-connect marks 24 -> 21
Changed lines of the file:
@@
 	7900 4900 6600 4900
 Wire Wire Line
-	6600 5000 7900 5000
+	6600 5000 6750 5000
 Wire Wire Line
 	7900 5100 6600 5100
@@
 	4950 5000 4950 6050
 Wire Wire Line
-	4950 6050 7900 6050
-Wire Wire Line
 	3700 3600 4000 3600
 Wire Wire Line
-	4000 3600 4000 6050
+	4000 3600 4000 4050
 Wire Wire Line
 	4000 6050 4950 6050
 Connection ~ 4950 6050
 Wire Wire Line
-	7900 950  7900 3050
+	7900 950  7900 2850
 Wire Wire Line
 	6200 2450 6200 2550
@@
 	3700 3700 3850 3700
 Wire Wire Line
-	3850 3700 3850 950
+	3850 3700 3850 3000
 Wire Wire Line
 	3850 950  4900 950
@@
 Wire Wire Line
 	3250 2450 4800 2450
-Wire Wire Line
-	5300 2450 5300 3400
-Wire Wire Line
-	5300 3400 3700 3400
-Wire Wire Line
-	3700 3500 5400 3500
-Wire Wire Line
-	5400 3500 5400 2450
-Wire Wire Line
-	3850 3700 7900 3700
 Connection ~ 3850 3700
 Wire Wire Line
-	7900 3900 7200 3900
+	7900 3900 7800 3900
 Wire Wire Line
 	7200 3900 7200 2550
@@
 NoConn ~ 5100 2450
 NoConn ~ 5200 2450
-NoConn ~ 5500 2450
-NoConn ~ 5600 2450
 NoConn ~ 5700 2450
 NoConn ~ 5800 2450
 NoConn ~ 5900 2450
 NoConn ~ 6000 2450
-NoConn ~ 2250 5850
+$Comp
+L Device:C C1
+U 1 1 5E9376D9
+P 7600 3100
+F 0 "C1" H 7715 3146 50  0000 L CNN
+F 1 "C" H 7715 3055 50  0000 L CNN
+F 2 "" H 7638 2950 50  0001 C CNN
+F 3 "~" H 7600 3100 50  0001 C CNN
+	1    7600 3100
+	1    0    0    -1
+$EndComp
+Wire Wire Line
+	7600 2950 7900 2950
+Connection ~ 7900 2950
+Wire Wire Line
+	7900 2950 7900 3050
+Wire Wire Line
+	7600 3250 7600 3300
+Wire Wire Line
+	7600 3300 7900 3300
+Connection ~ 7900 3300
+$Comp
+L Device:R R2
+U 1 1 5E93A593
+P 4000 3000
+F 0 "R2" H 4070 3046 50  0000 L CNN
+F 1 "R" H 4070 2955 50  0000 L CNN
+F 2 "" V 3930 3000 50  0001 C CNN
+F 3 "~" H 4000 3000 50  0001 C CNN
+	1    4000 3000
+	0    -1   -1   0
+$EndComp
+$Comp
+L Device:R R1
+U 1 1 5E93B25F
+P 4000 2750
+F 0 "R1" H 4070 2796 50  0000 L CNN
+F 1 "R" H 4070 2705 50  0000 L CNN
+F 2 "" V 3930 2750 50  0001 C CNN
+F 3 "~" H 4000 2750 50  0001 C CNN
+	1    4000 2750
+	0    -1   -1   0
+$EndComp
+Wire Wire Line
+	4950 4700 4950 4050
+Wire Wire Line
+	4950 4050 7350 4050
+Wire Wire Line
+	7350 4050 7350 2850
+Wire Wire Line
+	7350 2850 7900 2850
+Connection ~ 7900 2850
+Wire Wire Line
+	7900 2850 7900 2950
+Wire Wire Line
+	3850 3700 4150 3700
+Wire Wire Line
+	3700 3400 4250 3400
+Wire Wire Line
+	5300 3400 5300 2450
+Wire Wire Line
+	3700 3500 4350 3500
+Wire Wire Line
+	5400 3500 5400 2450
+Wire Wire Line
+	4950 4800 4850 4800
+Wire Wire Line
+	4850 4800 4850 3950
+Wire Wire Line
+	4850 3950 5600 3950
+Wire Wire Line
+	5600 3950 5600 2450
+Wire Wire Line
+	4950 4900 4750 4900
+Wire Wire Line
+	4750 4900 4750 3850
+Wire Wire Line
+	4750 3850 5500 3850
+Wire Wire Line
+	5500 3850 5500 2450
+Connection ~ 3850 2750
+Wire Wire Line
+	3850 2750 3850 950
+Connection ~ 3850 3000
+Wire Wire Line
+	3850 3000 3850 2750
+Wire Wire Line
+	4150 3000 4250 3000
+Wire Wire Line
+	4250 3000 4250 3400
+Connection ~ 4250 3400
+Wire Wire Line
+	4250 3400 5300 3400
+Wire Wire Line
+	4150 2750 4350 2750
+Wire Wire Line
+	4350 2750 4350 3500
+Connection ~ 4350 3500
+Wire Wire Line
+	4350 3500 5400 3500
+Wire Wire Line
+	6750 5000 6750 6050
+Wire Wire Line
+	4950 6050 6750 6050
+Connection ~ 6750 5000
+Wire Wire Line
+	6750 5000 7900 5000
+Connection ~ 6750 6050
+Wire Wire Line
+	6750 6050 7900 6050
+$Comp
+L Device:C C2
+U 1 1 5E953AE5
+P 4150 3900
+F 0 "C2" H 4265 3946 50  0000 L CNN
+F 1 "C" H 4265 3855 50  0000 L CNN
+F 2 "" H 4188 3750 50  0001 C CNN
+F 3 "~" H 4150 3900 50  0001 C CNN
+	1    4150 3900
+	1    0    0    -1
+$EndComp
+$Comp
+L Device:C C3
+U 1 1 5E956511
+P 7650 4200
+F 0 "C3" H 7765 4246 50  0000 L CNN
+F 1 "C" H 7765 4155 50  0000 L CNN
+F 2 "" H 7688 4050 50  0001 C CNN
+F 3 "~" H 7650 4200 50  0001 C CNN
+	1    7650 4200
+	0    -1   -1   0
+$EndComp
+Wire Wire Line
+	7500 4200 7500 3700
+Connection ~ 7500 3700
+Wire Wire Line
+	7500 3700 7900 3700
+Wire Wire Line
+	7800 4200 7800 3900
+Connection ~ 7800 3900
+Wire Wire Line
+	7800 3900 7200 3900
+Wire Wire Line
+	4150 3750 4150 3700
+Connection ~ 4150 3700
+Wire Wire Line
+	4150 3700 7500 3700
+Wire Wire Line
+	4150 4050 4000 4050
+Connection ~ 4000 4050
+Wire Wire Line
+	4000 4050 4000 6050
 $EndSCHEMATC

Commit message: added I2S removed C3 removed Reed switch
Parts:
- removed C3: C, symbol Device:C
- removed SW1: SW_Reed, symbol Switch:SW_Reed
- added R3: 4k7, symbol Device:R
- added U7: I2SSpringTerm, symbol ESP32~Waage:I2SSpringTerm
- C1, C2: value C -> 100nF
- R1, R2: value R -> 4k7
Connections:
- wire segments 83 -> 86
- no-connect marks 21 -> 18
Other:
- moved on the sheet: C1, C2, R1, R2

Commit message: Optocoupler Mounting holes
Parts:
- added C3, C4: 1uF, Capacitor_THT:C_Disc_D3.4mm_W2.1mm_P2.50mm, symbol Device:C
- added C?: 1uF, symbol Device:C
- added H1: SDA, symbol Mechanical:MountingHole_Pad
- added H10: 34, symbol Mechanical:MountingHole_Pad
- added H11: RXD, symbol Mechanical:MountingHole_Pad
- added H12: 35, symbol Mechanical:MountingHole_Pad
- added H13: 22, symbol Mechanical:MountingHole_Pad
- added H14: 19, symbol Mechanical:MountingHole_Pad
- added H15: 23, symbol Mechanical:MountingHole_Pad
- added H16: 27, symbol Mechanical:MountingHole_Pad
- added H17: 14, symbol Mechanical:MountingHole_Pad
- added H18: 12, symbol Mechanical:MountingHole_Pad
- added H19: 0, symbol Mechanical:MountingHole_Pad
- added H2: SDC, symbol Mechanical:MountingHole_Pad
- added H20: 13, symbol Mechanical:MountingHole_Pad
- added H21: 4, symbol Mechanical:MountingHole_Pad
- added H3: VCC, symbol Mechanical:MountingHole_Pad
- added H4: GND, symbol Mechanical:MountingHole_Pad
- added H5: 36, symbol Mechanical:MountingHole_Pad
- added H6: 39, symbol Mechanical:MountingHole_Pad
- added H7: 21, symbol Mechanical:MountingHole_Pad
- added H8: RST, symbol Mechanical:MountingHole_Pad
- added H9: TXD, symbol Mechanical:MountingHole_Pad
- added R4, R5: 680, symbol Device:R
- added R6, R7: 470, symbol Device:R
- added U8, U9: 4N35, Package_DIP:DIP-6_W7.62mm, symbol Isolator:4N35
- C1, C2: value 100nF -> 47uF; footprint (none) -> Capacitor_THT:C_Disc_D3.4mm_W2.1mm_P2.50mm
- R1, R2, R3: footprint (none) -> Resistor_THT:R_Axial_DIN0207_L6.3mm_D2.5mm_P10.16mm_Horizontal
- U1: footprint (none) -> ESP32 Waage:BME280_Socket
- U2: footprint (none) -> ESP32 Waage:TTGO_T8_Socket
- U3: footprint (none) -> ESP32 Waage:HX711_Socket
- U4: footprint (none) -> TerminalBlock_TE-Connectivity:TerminalBlock_TE_282834-2_1x02_P2.54mm_Horizontal
- U5, U7: footprint (none) -> TerminalBlock_TE-Connectivity:TerminalBlock_TE_282834-3_1x03_P2.54mm_Horizontal
- U6: footprint (none) -> TerminalBlock_TE-Connectivity:TerminalBlock_TE_282834-7_1x07_P2.54mm_Horizontal
Connections:
- wire segments 86 -> 130
- no-connect marks 18 -> 4
Other:
- moved on the sheet: C2, R1, R2

Commit message: removed optocouplers added LVC74...
Parts:
- removed R4, R5: 680, symbol Device:R
- removed R6, R7: 470, symbol Device:R
- removed U8, U9: 4N35, Package_DIP:DIP-6_W7.62mm, symbol Isolator:4N35
- added C6: 1uF, Capacitor_THT:C_Disc_D3.4mm_W2.1mm_P2.50mm, symbol Device:C
- added U8: SN74LVC1T45DBV, Package_TO_SOT_SMD:SOT-23-6, symbol Logic_LevelTranslator:SN74LVC1T45DBV
- gave numbers to parts that had none: 1
Connections:
- wire segments 130 -> 126
- no-connect marks 4 -> 2
Other:
- moved on the sheet: C1, C2, C3, C4, C5, R1, R2, R3

Commit message: added switch rearranged stuff
Parts:
- removed C6: 1uF, Capacitor_THT:C_Disc_D3.4mm_W2.1mm_P2.50mm, symbol Device:C
- removed H1: SDA, symbol Mechanical:MountingHole_Pad
- removed H10: 34, symbol Mechanical:MountingHole_Pad
- removed H11: RXD, symbol Mechanical:MountingHole_Pad
- removed H12: 35, symbol Mechanical:MountingHole_Pad
- removed H13: 22, symbol Mechanical:MountingHole_Pad
- removed H14: 19, symbol Mechanical:MountingHole_Pad
- removed H15: 23, symbol Mechanical:MountingHole_Pad
- removed H16: 27, symbol Mechanical:MountingHole_Pad
- removed H17: 14, symbol Mechanical:MountingHole_Pad
- removed H18: 12, symbol Mechanical:MountingHole_Pad
- removed H19: 0, symbol Mechanical:MountingHole_Pad
- removed H2: SDC, symbol Mechanical:MountingHole_Pad
- removed H20: 13, symbol Mechanical:MountingHole_Pad
- removed H21: 4, symbol Mechanical:MountingHole_Pad
- removed H3: VCC, symbol Mechanical:MountingHole_Pad
- removed H4: GND, symbol Mechanical:MountingHole_Pad
- removed H5: 36, symbol Mechanical:MountingHole_Pad
- removed H6: 39, symbol Mechanical:MountingHole_Pad
- removed H7: 21, symbol Mechanical:MountingHole_Pad
- removed H8: RST, symbol Mechanical:MountingHole_Pad
- removed H9: TXD, symbol Mechanical:MountingHole_Pad
- added SW1: SW_SPST, Button_Switch_THT:SW_CuK_JS202011CQN_DPDT_Straight, symbol Switch:SW_SPST
- added TP1, TP10, TP11, TP12, TP13, TP14, TP15, TP16, TP17, TP2, TP3, TP4, TP5, TP6, TP7, TP8, TP9: TestPoint, TestPoint:TestPoint_THTPad_D2.0mm_Drill1.0mm, symbol Connector:TestPoint
- added U9: I2CSpringTerm, TerminalBlock_TE-Connectivity:TerminalBlock_TE_282834-4_1x04_P2.54mm_Horizontal, symbol ESP32~Waage:I2CSpringTerm
- C1: renamed from C3; footprint Capacitor_THT:C_Disc_D3.4mm_W2.1mm_P2.50mm -> Capacitor_SMD:C_0805_2012Metric_Pad1.15x1.40mm_HandSolder
- C2: renamed from C1; footprint Capacitor_THT:C_Disc_D3.4mm_W2.1mm_P2.50mm -> Capacitor_SMD:C_0805_2012Metric_Pad1.15x1.40mm_HandSolder
- C3: renamed from C2; footprint Capacitor_THT:C_Disc_D3.4mm_W2.1mm_P2.50mm -> Capacitor_SMD:C_0805_2012Metric_Pad1.15x1.40mm_HandSolder
- C4: renamed from C5; footprint (none) -> Capacitor_SMD:C_0805_2012Metric_Pad1.15x1.40mm_HandSolder
- C5: renamed from C4; footprint Capacitor_THT:C_Disc_D3.4mm_W2.1mm_P2.50mm -> Capacitor_SMD:C_0805_2012Metric_Pad1.15x1.40mm_HandSolder
- R1: renamed from R3; footprint Resistor_THT:R_Axial_DIN0207_L6.3mm_D2.5mm_P10.16mm_Horizontal -> Resistor_SMD:R_0805_2012Metric_Pad1.15x1.40mm_HandSolder
- R2: renamed from R1; footprint Resistor_THT:R_Axial_DIN0207_L6.3mm_D2.5mm_P10.16mm_Horizontal -> Resistor_SMD:R_0805_2012Metric_Pad1.15x1.40mm_HandSolder
- R3: renamed from R2; footprint Resistor_THT:R_Axial_DIN0207_L6.3mm_D2.5mm_P10.16mm_Horizontal -> Resistor_SMD:R_0805_2012Metric_Pad1.15x1.40mm_HandSolder
- U8: renamed from U7; footprint TerminalBlock_TE-Connectivity:TerminalBlock_TE_282834-3_1x03_P2.54mm_Horizontal -> TerminalBlock_TE-Connectivity:TerminalBlock_TE_282834-6_1x06_P2.54mm_Horizontal
- renumbered U4 to U1, U8 to U2, U2 to U3, U3 to U4, U1 to U5, U5 to U7
Connections:
- net labels added: +3.3V
- wire segments 126 -> 115
Other:
- moved on the sheet: C1, C2, C3, C4, C5, R1, R2, R3, U2

Commit message: new schema layout
Parts:
- removed TP1, TP10, TP11, TP12, TP13, TP14, TP15, TP16, TP17, TP2, TP3, TP4, TP5, TP6, TP7, TP8, TP9: TestPoint, TestPoint:TestPoint_THTPad_D2.0mm_Drill1.0mm, symbol Connector:TestPoint
- removed U1: SupplSpringTerm, TerminalBlock_TE-Connectivity:TerminalBlock_TE_282834-2_1x02_P2.54mm_Horizontal, symbol ESP32~Waage:SupplSpringTerm
- removed U5: BME280Socket, ESP32 Waage:BME280_Socket, symbol ESP32~Waage:BME280Socket
- removed U6: HX711SpringTerm, TerminalBlock_TE-Connectivity:TerminalBlock_TE_282834-7_1x07_P2.54mm_Horizontal, symbol ESP32~Waage:HX711SpringTerm
- removed U7: DS18B20SpringTerm, TerminalBlock_TE-Connectivity:TerminalBlock_TE_282834-3_1x03_P2.54mm_Horizontal, symbol ESP32~Waage:DS18B20SpringTerm
- removed U8: I2SSpringTerm, TerminalBlock_TE-Connectivity:TerminalBlock_TE_282834-6_1x06_P2.54mm_Horizontal, symbol ESP32~Waage:I2SSpringTerm
- removed U9: I2CSpringTerm, TerminalBlock_TE-Connectivity:TerminalBlock_TE_282834-4_1x04_P2.54mm_Horizontal, symbol ESP32~Waage:I2CSpringTerm
- added J1: Ext. Power Supply 5V, symbol Connector:Conn_01x02_Female
- added J10: I2S Terminal, symbol Connector:Conn_01x06_Female
- added J11: Ext. BME280, symbol Connector:Conn_01x06_Female
- added J12: Int. BME280, symbol Connector:Conn_01x06_Female
- added J2: spare, Connector_PinHeader_2.54mm:PinHeader_1x08_P2.54mm_Vertical, symbol Connector:Conn_01x08_Female
- added J3: spare, Connector_PinHeader_2.54mm:PinHeader_1x02_P2.54mm_Vertical, symbol Connector:Conn_01x02_Female
- added J4: 5V spare, Connector_PinSocket_2.54mm:PinSocket_1x02_P2.54mm_Vertical, symbol Connector:Conn_01x02_Female
- added J5: 3.3V spare, Connector_PinSocket_2.54mm:PinSocket_1x02_P2.54mm_Vertical, symbol Connector:Conn_01x02_Female
- added J6: spare, Connector_PinHeader_2.54mm:PinHeader_1x05_P2.54mm_Vertical, symbol Connector:Conn_01x05_Female
- added J7: spare, Connector_PinSocket_2.54mm:PinSocket_1x02_P2.54mm_Vertical, symbol Connector:Conn_01x02_Female
- added J8: Scale Terminal, symbol Connector:Conn_01x07_Female
- added J9: DS18B20 Term., symbol Connector:Conn_01x03_Female
- renumbered C2 to C1, C1 to C2, R3 to R1, R1 to R3, U2 to U1, U3 to U2, U4 to U3
Connections:
- net labels added: 21, 32, 33, 3V3, CSB, Data, L_R, SCK, SD, SDA, SDC, SDO, WS
- wire segments 115 -> 121
Other:
- moved on the sheet: C1, C2, C3, C4, C5, R1, R2, R3, SW1, U1

Commit message: redesign of schema added various 3D models PCB
Parts:
- added C6: 1uF, Capacitor_SMD:C_0805_2012Metric_Pad1.15x1.40mm_HandSolder, symbol Device:C
- J10, J11: footprint (none) -> ESP32 Waage:PhoenixContact_FFKDSV_254_6_pol
- J12: footprint (none) -> ESP32 Waage:BME280_Socket
- J2: renamed from J1; footprint (none) -> ESP32 Waage:PhoenixContact_FFKDSV_254_2_pol
- J7: footprint Connector_PinSocket_2.54mm:PinSocket_1x02_P2.54mm_Vertical -> Connector_PinHeader_2.54mm:PinHeader_1x02_P2.54mm_Vertical
- J8: footprint (none) -> ESP32 Waage:PhoenixContact_FFKDSV_254_7_pol
- J9: footprint (none) -> ESP32 Waage:PhoenixContact_FFKDSV_254_3_pol
- renumbered J5 to J1, J2 to J3, J3 to J4, J4 to J5
Connections:
- net labels added: +3V3, +5VL
- net labels removed: +3.3V, 3V3, CSB, Data, L_R, SDO
- wire segments 121 -> 128
Other:
- note added: "3V3"
- note added: "CSB"
- note added: "Data"
- note added: "GND"
- note added: "L/R"
- note added: "SCK"
- note added: "SD"
- note added: "SDA"
- note added: "SDC"
- note added: "SDO"
- note added: "WS"
- moved on the sheet: J1, J11, J12, R1, R2

Commit message: change from 2,54 terminals to 3,81 because of availability removed internal I2C & BME280 added mounting holes
Parts:
- removed C6: 1uF, Capacitor_SMD:C_0805_2012Metric_Pad1.15x1.40mm_HandSolder, symbol Device:C
- removed J11: Ext. BME280, ESP32 Waage:PhoenixContact_FFKDSV_254_6_pol, symbol Connector:Conn_01x06_Female
- removed J12: Int. BME280, ESP32 Waage:BME280_Socket, symbol Connector:Conn_01x06_Female
- added J11: I2C Terminal, ESP32 Waage:PhoenixContact_FFKDSV_381_4_pol, symbol Connector:Conn_01x04_Female
- J10: footprint ESP32 Waage:PhoenixContact_FFKDSV_254_6_pol -> ESP32 Waage:PhoenixContact_FFKDSV_381_6_pol
- J2: footprint ESP32 Waage:PhoenixContact_FFKDSV_254_2_pol -> ESP32 Waage:PhoenixContact_FFKDSV_381_2_pol
- J8: footprint ESP32 Waage:PhoenixContact_FFKDSV_254_7_pol -> ESP32 Waage:PhoenixContact_FFKDSV_381_7_pol
- J9: footprint ESP32 Waage:PhoenixContact_FFKDSV_254_3_pol -> ESP32 Waage:PhoenixContact_FFKDSV_381_3_pol
Connections:
- wire segments 128 -> 106
- no-connect marks 2 -> 0
Other:
- note removed: "CSB"
- note removed: "SDO"
- moved on the sheet: C5, R1, R2, R3
